File: hw/encoder/encoderBoard/encoderBoard.sch (KiCad schematic (older format))
At the start: 5 parts, among them J1 Conn_01x03, U1 MH253

Commit message: Swap pinhead pinout, add GND polygon to bottom
Connections:
- net VCC: now also J1.2 (Pin_2); no longer J1.3 (Pin_3)
- net at C2.1, R1.2, U1.2 (OUT): now also J1.3 (Pin_3); no longer J1.2 (Pin_2)
Changed lines of the file:
@@
 Wire Wire Line
 	4550 2650 5050 2650
-Wire Wire Line
-	5050 2650 5050 3050
-Wire Wire Line
-	5050 3050 5200 3050
 Connection ~ 4550 2650
-Wire Wire Line
-	4550 3150 5200 3150
 Wire Wire Line
 	4550 3600 5050 3600
 Wire Wire Line
 	5050 3600 5050 3250
+Connection ~ 4550 3600
+Wire Wire Line
+	5050 3150 5200 3150
+Wire Wire Line
+	5050 2650 5050 3150
 Wire Wire Line
 	5050 3250 5200 3250
-Connection ~ 4550 3600
+Wire Wire Line
+	4950 3150 4950 3050
+Wire Wire Line
+	4950 3050 5200 3050
+Wire Wire Line
+	4550 3150 4950 3150
 $EndSCHEMATC
