File: hw/tachometer/tachometer.kicad_pcb (KiCad board)
At the start: 2 copper layers, 91.4 x 50 mm, 56 parts, among them J1 Pmod JA, J2 Pmod JB, J3 Pmod JC, J4 Pmod JD, J5 HallSensor1, J6 HallSensor2, Q1 BC817, Q2 BC817, Q3 BC817, Q4 BC817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

Commit message: Final routing boards
Parts:
- removed D7, D8: LED, LED_THT:LED_D5.0mm
- removed R28, R29: 220, Resistor_SMD:R_0603_1608Metric_Pad0.98x0.95mm_HandSolder
- added R30: 220, Resistor_SMD:R_0603_1608Metric_Pad0.98x0.95mm_HandSolder, B.Cu at (105.2, 139.0)
- added R31: 220, Resistor_SMD:R_0603_1608Metric_Pad0.98x0.95mm_HandSolder, B.Cu at (107.6, 139.0)
- added R32: 220, Resistor_SMD:R_0603_1608Metric_Pad0.98x0.95mm_HandSolder, B.Cu at (110.2, 139.1)
- moved R3 14.2 mm to (149.2, 139.0)
- moved R4 12.6 mm to (152.7, 139.0)
- moved R10 7.18 mm to (161.2, 139.0)
- moved R2 7.15 mm to (138.3, 139.1)
- moved R9 5.65 mm to (157.8, 139.0)
- moved R5 5.59 mm to (156.1, 139.0)
- moved R11 5.46 mm to (132.6, 139.1)
- moved R26 5.21 mm to (134.5, 139.1)
- moved R7 5.02 mm to (150.9, 139.0)
- moved R17 4.19 mm to (128.8, 139.1)
- moved R21 4.07 mm to (130.7, 139.1)
- moved R8 3.62 mm to (154.4, 139.0)
- moved R14 3.56 mm to (136.4, 139.1)
- moved R6 0.39 mm to (159.5, 139.0)
- moved C1 0.09 mm to (130.8, 133.7)
Connections:
- C1 pad 2: G13 -> Net-(C1-Pad2)
- C2 pad 2: B11 -> Net-(C2-Pad2)
- C3 pad 2: A11 -> Net-(C3-Pad2)
- R1 pad 2: G13 -> Net-(C1-Pad2)
- R13 pad 2: B11 -> Net-(C2-Pad2)
- R16 pad 2: A11 -> Net-(C3-Pad2)
- SW1 pad 1: G13 -> Net-(C1-Pad2)
- SW2 pad 1: B11 -> Net-(C2-Pad2)
- SW3 pad 1: A11 -> Net-(C3-Pad2)
Routing:
- net VCC: track 0.00 -> 235.0 mm
- net K16: track 0.00 -> 90.0 mm
- net A18: track 0.00 -> 81.5 mm
- net B18: track 0.00 -> 74.0 mm
- net D12: track 0.00 -> 70.8 mm
- net D13: track 0.00 -> 66.1 mm
- net Net-(C3-Pad2): track 0.00 -> 62.0 mm, vias 0 -> 1
- net Net-(C2-Pad2): track 0.00 -> 49.6 mm, vias 0 -> 1
- net Net-(Q3-Pad1): track 0.00 -> 49.5 mm, vias 0 -> 2
- net Net-(Q4-Pad1): track 0.00 -> 47.0 mm, vias 0 -> 2
- net Net-(C1-Pad2): track 0.00 -> 37.0 mm, vias 0 -> 1
- net H2: track 0.00 -> 36.5 mm
- net Net-(D1-Pad12): track 0.00 -> 35.5 mm, vias 0 -> 1
- net Net-(D1-Pad15): track 0.00 -> 35.0 mm, vias 0 -> 1
- net Net-(D1-Pad16): track 0.00 -> 34.8 mm, vias 0 -> 1
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- added copper zone on B.Cu, net GND
- added copper zone on F.Cu, net GND
Other:
- board text added: "->"
- board text added: "<-"
- board text added: "Calories"
- board text added: "DATA"
- board text added: "Distance"
- board text added: "GND"
- board text added: "OK"
- board text added: "Speed"
- board text added: "TachometerBoard BPC-DE1 project 05/2021"
- board text added: "Time"
- board text added: "Trip"
- board text added: "VCC"
