File: hw/tachometer/tachometer.sch (KiCad schematic (older format))
At the start: 54 parts, among them J1 Pmod JA, J2 Pmod JB, J3 Pmod JC, J4 Pmod JD, J5 HallSensor1, J6 HallSensor2, Q1 BC817, Q2 BC817, Q3 BC817, Q4 BC817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

Commit message: Final routing boards
Parts:
- removed D7, D8: LED, LED_THT:LED_D5.0mm, symbol Device:LED
- removed R28, R29: 220, Resistor_SMD:R_0603_1608Metric_Pad0.98x0.95mm_HandSolder, symbol Device:R
- added R30, R31, R32: 220, Resistor_SMD:R_0603_1608Metric_Pad0.98x0.95mm_HandSolder, symbol Device:R
Connections:
- net A11: now also R32.2; no longer C3.2, R16.2, SW3.1, SW3.3
- net B11: now also R31.2; no longer C2.2, R13.2, SW2.1, SW2.3
- net G13: now also R30.2; no longer C1.2, R1.2, SW1.1, SW1.3
- new net: C3.2, R16.2, R32.1, SW3.1, SW3.3
- new net: C2.2, R13.2, R31.1, SW2.1, SW2.3
- new net: C1.2, R1.2, R30.1, SW1.1, SW1.3
Other:
- note removed: "Fitness"
- moved on the sheet: C1, C2, C3, R1, R13, R16, SW1, SW2, SW3
